Commit message: Modified floor & robot on gazebo

File: ros_ws/install/line_follower/share/line_follower/urdf/robot.urdf (robot description, URDF)
Before this commit: robot line_robot, 4 links, 3 joints
Links:
- removed link camera_link
- link left_wheel: mass None -> 0.2
- link right_wheel: mass None -> 0.2
Joints:
- removed joint camera_joint
- joint left_wheel_joint: axis 0 0 1 -> 0 1 0; origin xyz=0 0.08 -0.03 rpy=1.5707 0 0 -> xyz=0 0.08 0.03
- joint right_wheel_joint: axis 0 0 1 -> 0 1 0; origin xyz=0 -0.08 -0.03 rpy=1.5707 0 0 -> xyz=0 -0.08 0.03

Commit message: Modified all nodes files

File: ros_ws/install/line_follower/share/line_follower/urdf/robot.urdf (robot description, URDF)
Before this commit: robot line_robot, 3 links, 2 joints
Links:
- added link ir_center
- added link ir_left
- added link ir_right
Joints:
- added joint ir_center_joint: type fixed, parent base_link, child ir_center, origin xyz=0.08 0.0 0.01
- added joint ir_left_joint: type fixed, parent base_link, child ir_left, origin xyz=0.08 0.03 0.01
- added joint ir_right_joint: type fixed, parent base_link, child ir_right, origin xyz=0.08 -0.03 0.01
